File: SparkFun Load Sensor Combinator.brd (EAGLE design)
At the start: 27.9 x 17.8 mm, 15 parts, among them J1 RJ11-6PTH

Commit message: Added feedback from Eng review
Match 5-pin connector on breakout. Add yellow pin with NC. Add note to
schematic describing that 4 sensors create one load cell.
Parts:
- removed J1: RJ11-6PTH, SparkFun-Connectors:RJ11-6
- removed JP6: (no value), SparkFun-Connectors:SCREWTERMINAL-3.5MM-4
- removed U$1: RJ45-8PTH, SparkFun-Connectors:RJ45-8
- FRAME1: value FRAME-LETTER -> (none)
- JP3: value (none) -> LL; device SparkFun-Connectors:1X04 -> SparkFun-Connectors:1X03
- JP4: value LL -> LR
- JP5: value LR -> (none); device SparkFun-Connectors:1X03 -> SparkFun-Connectors:1X05
- moved JP5 18.0 mm to (8.89, 16.5), turned to 0 degrees
- moved FRAME1 15.8 mm to (-12.7, -11.4)
- moved JP3 14.2 mm to (16.5, 3.81), turned to 90 degrees
- moved JP4 5.08 mm to (21.6, 3.81)
Connections:
- net A+: now also JP3.3, JP5.3; no longer JP3.4, JP4.3
- net A-: now also JP5.4; no longer JP3.3
- net E+: now also JP4.3, JP5.1; no longer JP3.1, JP5.3
- net E-: now also JP5.2; no longer JP3.2
- net N$1: now also JP4.1; no longer JP5.1
- net N$2: now also JP3.1; no longer JP4.1
- net N$3: now also JP3.2; no longer JP5.2
Routing:
- net A-: track 9.20 -> 15.2 mm, vias 0 -> 1
- net E-: track 11.7 -> 10.5 mm
- net A+: track 8.15 -> 8.67 mm
- net E+: track 17.6 -> 18.1 mm
Other:
- board text added: "SLD"
- board text added: "YLW"
- board text added: "v02"
- board text removed: "N. Seidle"
- board text removed: "V10"
Changed lines of the file:
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@@
 <?xml version="1.0" encoding="utf-8"?>
 <!DOCTYPE eagle SYSTEM "eagle.dtd">
-<eagle version="7.1.0">
+<eagle version="7.2.0">
 <drawing>
 <settings>
@@
 <layer number="47" name="Measures" color="7" fill="1" visible="no" active="yes"/>
 <layer number="48" name="Document" color="7" fill="1" visible="no" active="yes"/>
-<layer number="49" name="Reference" color="7" fill="1" visible="no" active="yes"/>
+<layer number="49" name="Reference" color="7" fill="1" visible="yes" active="yes"/>
 <layer number="50" name="dxf" color="7" fill="1" visible="no" active="no"/>
 <layer number="51" name="tDocu" color="6" fill="1" visible="yes" active="yes"/>
@@
 <wire x1="27.94" y1="0" x2="0" y2="0" width="0.2032" layer="20"/>
 <wire x1="0" y1="0" x2="0" y2="17.78" width="0.2032" layer="20"/>
-<text x="15.875" y="11.557" size="1.27" layer="21" font="vector" ratio="15" rot="R90">GRN</text>
+<text x="17.145" y="11.557" size="1.27" layer="21" font="vector" ratio="15" rot="R90">GRN</text>
 <text x="22.225" y="0.635" size="1.27" layer="22" font="vector" ratio="15" rot="MR0">Load Combinator</text>
-<text x="13.335" y="11.557" size="1.27" layer="21" font="vector" ratio="15" rot="R90">BLK</text>
-<text x="18.415" y="11.557" size="1.27" layer="21" font="vector" ratio="15" rot="R90">WHT</text>
-<text x="10.795" y="11.557" size="1.27" layer="21" font="vector" ratio="15" rot="R90">RED</text>
-<text x="14.605" y="12.192" size="1.27" layer="22" font="vector" ratio="15" rot="MR90">A+</text>
-<text x="17.145" y="12.192" size="1.27" layer="22" font="vector" ratio="15" rot="MR90">A-</text>
-<text x="12.065" y="12.192" size="1.27" layer="22" font="vector" ratio="15" rot="MR90">E-</text>
-<text x="9.525" y="12.192" size="1.27" layer="22" font="vector" ratio="15" rot="MR90">E+</text>
-<text x="2.54" y="10.541" size="1.27" layer="16" font="vector" ratio="20" rot="MR270">V10</text>
+<text x="12.065" y="11.557" size="1.27" layer="21" font="vector" ratio="15" rot="R90">BLK</text>
+<text x="14.605" y="11.557" size="1.27" layer="21" font="vector" ratio="15" rot="R90">WHT</text>
+<text x="9.525" y="11.557" size="1.27" layer="21" font="vector" ratio="15" rot="R90">RED</text>
+<text x="17.145" y="15.24" size="1.27" layer="22" font="vector" ratio="15" rot="MR270">A+</text>
+<text x="14.605" y="15.24" size="1.27" layer="22" font="vector" ratio="15" rot="MR270">A-</text>
+<text x="12.065" y="15.24" size="1.27" layer="22" font="vector" ratio="15" rot="MR270">E-</text>
+<text x="9.525" y="15.24" size="1.27" layer="22" font="vector" ratio="15" rot="MR270">E+</text>
 <text x="5.334" y="0.508" size="1.27" layer="21" font="vector" ratio="15">UL</text>
 <text x="10.414" y="0.508" size="1.27" layer="21" font="vector" ratio="15">UR</text>
 <text x="15.494" y="0.635" size="1.27" layer="21" font="vector" ratio="15">LL</text>
 <text x="20.574" y="0.635" size="1.27" layer="21" font="vector" ratio="15">LR</text>
-<text x="30.48" y="-21.59" size="1.778" layer="51" font="vector" ratio="15">N. Seidle</text>
 <text x="2.413" y="6.477" size="1.27" layer="21" font="vector" ratio="15" rot="R90">Load</text>
 <text x="12.446" y="10.414" size="1.27" layer="22" font="vector" ratio="15" rot="MR0">UR</text>
@@
 <text x="8.255" y="5.461" size="1.778" layer="21" font="vector" ratio="15">W</text>
 <text x="8.255" y="7.874" size="1.778" layer="21" font="vector" ratio="15">R</text>
+<text x="26.289" y="11.43" size="1.778" layer="16" font="vector" ratio="15" rot="MR270">v02</text>
+<text x="19.685" y="11.557" size="1.27" layer="21" font="vector" ratio="15" rot="R90">YLW</text>
+<text x="19.685" y="15.24" size="1.27" layer="22" font="vector" ratio="15" rot="MR270">SLD</text>
 </plain>
 <attributes>
@@
 <elements>
 <element name="U$7" library="SparkFun-Aesthetics" package="OSHW-LOGO-S" value="OSHW-LOGOS" x="6.35" y="15.24" rot="MR0"/>
-<element name="FRAME1" library="SparkFun-Aesthetics" package="CREATIVE_COMMONS" value="FRAME-LETTER" x="-0.65105625" y="-21.59"/>
 <element name="STANDOFF1" library="SparkFun-Electromechanical" package="STAND-OFF" value="STAND-OFF" x="2.54" y="2.54"/>
 <element name="STANDOFF2" library="SparkFun-Electromechanical" package="STAND-OFF" value="STAND-OFF" x="25.4" y="2.54"/>
 <element name="STANDOFF3" library="SparkFun-Electromechanical" package="STAND-OFF" value="STAND-OFF" x="2.54" y="15.24"/>
 <element name="STANDOFF4" library="SparkFun-Electromechanical" package="STAND-OFF" value="STAND-OFF" x="25.4" y="15.24"/>
-<element name="JP3" library="SparkFun-Connectors" package="1X04" value="" x="10.16" y="16.51"/>
 <element name="LOGO3" library="SparkFun-Aesthetics" package="SFE_LOGO_FLAME_.1" value="SFE_LOGO_FLAME.1_INCH" x="20.701" y="13.716"/>
 <element name="JP1" library="SparkFun-Connectors" package="1X03" value="UL" x="6.35" y="3.81" rot="R90"/>
 <element name="JP2" library="SparkFun-Connectors" package="1X03" value="UR" x="11.43" y="3.81" rot="R90"/>
-<element name="JP4" library="SparkFun-Connectors" package="1X03" value="LL" x="16.51" y="3.81" rot="R90"/>
-<element name="JP5" library="SparkFun-Connectors" package="1X03" value="LR" x="21.59" y="3.81" rot="R90"/>
-<element name="J1" library="SparkFun-Connectors" package="RJ11-6" value="RJ11-6PTH" x="-11.43" y="22.86" rot="R180"/>
-<element name="U$1" library="SparkFun-Connectors" package="RJ45-8" value="RJ45-8PTH" x="-33.02" y="22.86" rot="R180"/>
-<element name="JP6" library="SparkFun-Connectors" package="SCREWTERMINAL-3.5MM-4" value="" x="8.89" y="22.86"/>
+<element name="JP3" library="SparkFun-Connectors" package="1X03" value="LL" x="16.51" y="3.81" rot="R90"/>
+<element name="JP4" library="SparkFun-Connectors" package="1X03" value="LR" x="21.59" y="3.81" rot="R90"/>
+<element name="FRAME1" library="SparkFun-Aesthetics" package="CREATIVE_COMMONS" value="" x="-12.7" y="-11.43">
+<attribute name="VERSION" value="v01" x="-12.7" y="-11.43" size="1.778" layer="27" font="vector" ratio="15" display="off"/>
+<attribute name="DESIGNER" value="N. Seidle" x="-12.7" y="-11.43" size="1.778" layer="27" font="vector" ratio="15" display="off"/>
+</element>
+<element name="JP5" library="SparkFun-Connectors" package="1X05" value="" x="8.89" y="16.51"/>
 </elements>
 <signals>
@@
 </signal>
 <signal name="N$1">
-<contactref element="JP5" pad="1"/>
+<contactref element="JP4" pad="1"/>
 <contactref element="JP2" pad="1"/>
 <wire x1="21.59" y1="3.81" x2="21.59" y2="2.54" width="0.508" layer="16"/>
@@
 </signal>
 <signal name="N$2">
-<contactref element="JP4" pad="1"/>
+<contactref element="JP3" pad="1"/>
 <contactref element="JP1" pad="1"/>
 <wire x1="6.35" y1="3.81" x2="6.35" y2="2.54" width="0.508" layer="1"/>
@@
 </signal>
 <signal name="N$3">
-<contactref element="JP5" pad="2"/>
 <contactref element="JP4" pad="2"/>
+<contactref element="JP3" pad="2"/>
 <wire x1="21.59" y1="6.35" x2="16.51" y2="6.35" width="0.508" layer="1"/>
 </signal>
@@
 </signal>
 <signal name="E+">
-<contactref element="JP5" pad="3"/>
-<contactref element="JP3" pad="1"/>
-<wire x1="10.16" y1="16.51" x2="10.16" y2="13.97" width="0.508" layer="16"/>
-<wire x1="10.16" y1="13.97" x2="11.43" y2="12.7" width="0.508" layer="16"/>
+<contactref element="JP4" pad="3"/>
 <wire x1="11.43" y1="12.7" x2="20.32" y2="12.7" width="0.508" layer="16"/>
 <wire x1="20.32" y1="12.7" x2="21.59" y2="11.43" width="0.508" layer="16"/>
 <wire x1="21.59" y1="11.43" x2="21.59" y2="8.89" width="0.508" layer="16"/>
+<contactref element="JP5" pad="1"/>
+<wire x1="11.43" y1="12.7" x2="8.89" y2="15.24" width="0.508" layer="16"/>
+<wire x1="8.89" y1="15.24" x2="8.89" y2="16.51" width="0.508" layer="16"/>
 </signal>
 <signal name="A+">
-<contactref element="JP4" pad="3"/>
-<contactref element="JP3" pad="4"/>
-<wire x1="17.78" y1="16.51" x2="17.78" y2="11.43" width="0.508" layer="1"/>
-<wire x1="17.78" y1="11.43" x2="16.51" y2="10.16" width="0.508" layer="1"/>
-<wire x1="16.51" y1="10.16" x2="16.51" y2="8.89" width="0.508" layer="1"/>
+<contactref element="JP3" pad="3"/>
+<contactref element="JP5" pad="3"/>
+<wire x1="16.51" y1="8.89" x2="16.51" y2="11.43" width="0.508" layer="1"/>
+<wire x1="16.51" y1="11.43" x2="13.97" y2="13.97" width="0.508" layer="1"/>
+<wire x1="13.97" y1="13.97" x2="13.97" y2="16.51" width="0.508" layer="1"/>
 </signal>
 <signal name="A-">
 <contactref element="JP2" pad="3"/>
-<contactref element="JP3" pad="3"/>
-<wire x1="15.24" y1="16.51" x2="15.24" y2="13.97" width="0.508" layer="1"/>
-<wire x1="15.24" y1="13.97" x2="11.43" y2="10.16" width="0.508" layer="1"/>
-<wire x1="11.43" y1="10.16" x2="11.43" y2="8.89" width="0.508" layer="1"/>
+<contactref element="JP5" pad="4"/>
+<wire x1="11.43" y1="8.89" x2="13.335" y2="10.795" width="0.508" layer="16"/>
+<wire x1="13.335" y1="10.795" x2="19.05" y2="10.795" width="0.508" layer="16"/>
+<via x="19.05" y="10.795" extent="1-16" drill="0.508"/>
+<wire x1="19.05" y1="10.795" x2="19.05" y2="12.7" width="0.508" layer="1"/>
+<wire x1="19.05" y1="12.7" x2="16.51" y2="15.24" width="0.508" layer="1"/>
+<wire x1="16.51" y1="15.24" x2="16.51" y2="16.51" width="0.508" layer="1"/>
 </signal>
 <signal name="E-">
-<contactref element="JP3" pad="2"/>
 <contactref element="JP1" pad="3"/>
-<wire x1="12.7" y1="16.51" x2="12.7" y2="13.97" width="0.508" layer="1"/>
-<wire x1="12.7" y1="13.97" x2="10.16" y2="11.43" width="0.508" layer="1"/>
-<wire x1="10.16" y1="11.43" x2="7.62" y2="11.43" width="0.508" layer="1"/>
+<wire x1="8.89" y1="11.43" x2="7.62" y2="11.43" width="0.508" layer="1"/>
 <wire x1="7.62" y1="11.43" x2="6.35" y2="10.16" width="0.508" layer="1"/>
 <wire x1="6.35" y1="10.16" x2="6.35" y2="8.89" width="0.508" layer="1"/>
+<contactref element="JP5" pad="2"/>
+<wire x1="8.89" y1="11.43" x2="11.43" y2="13.97" width="0.508" layer="1"/>
+<wire x1="11.43" y1="13.97" x2="11.43" y2="16.51" width="0.508" layer="1"/>
 </signal>
 </signals>
