File: SparkFun Load Sensor Combinator.sch (EAGLE design)
At the start: 15 parts, among them J1 RJ11-6PTH

Commit message: Added feedback from Eng review
Match 5-pin connector on breakout. Add yellow pin with NC. Add note to
schematic describing that 4 sensors create one load cell.
Parts:
- removed J1: RJ11-6PTH, SparkFun-Connectors:RJ11-6PTH
- removed JP6: (no value), SparkFun-Connectors:M04SCREW
- removed U$1: RJ45-8PTH, SparkFun-Connectors:RJ45-8PTH
- FRAME1: value FRAME-LETTER -> (none); DESIGNER (none) -> N. Seidle
- JP3: value (none) -> LL; device SparkFun-Connectors:M04PTH -> SparkFun-Connectors:M03PTH
- JP4: value LL -> LR
- JP5: value LR -> (none); device SparkFun-Connectors:M03PTH -> SparkFun-Connectors:M05PTH
Connections:
- net A+: now also JP3.3, JP5.3; no longer JP3.4, JP4.3
- net A-: now also JP5.4; no longer JP3.3
- net E+: now also JP4.3, JP5.1; no longer JP3.1, JP5.3
- net E-: now also JP5.2; no longer JP3.2
- net N$1: now also JP4.1; no longer JP5.1
- net N$2: now also JP3.1; no longer JP4.1
- net N$3: now also JP3.2; no longer JP5.2
Other:
- note added: "4 load sensors combine to create one load cell"
- note added: "Intentionally not-connected to create telescoping shield."
- note added: "Shield"
- note added: "Yellow"
- note removed: "N. Seidle"
- moved on the sheet: JP4
Changed lines of the file:
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@@
 <?xml version="1.0" encoding="utf-8"?>
 <!DOCTYPE eagle SYSTEM "eagle.dtd">
-<eagle version="7.1.0">
+<eagle version="7.2.0">
 <drawing>
 <settings>
@@
 <layer number="254" name="cooling" color="7" fill="1" visible="no" active="yes"/>
 </layers>
-<schematic xreflabel="%F%N/%S.%C%R" xrefpart="/%S.%C%R">
+<schematic xreflabel="%F%N/%S" xrefpart="/%S.%C%R">
 <attributes>
 </attributes>
@@
 </classes>
 <parts>
-<part name="FRAME1" library="SparkFun-Aesthetics" deviceset="FRAME-LETTER" device=""/>
 <part name="U$7" library="SparkFun-Aesthetics" deviceset="OSHW-LOGO" device="S"/>
 <part name="STANDOFF1" library="SparkFun-Electromechanical" deviceset="STAND-OFF" device=""/>
@@
 <part name="STANDOFF3" library="SparkFun-Electromechanical" deviceset="STAND-OFF" device=""/>
 <part name="STANDOFF4" library="SparkFun-Electromechanical" deviceset="STAND-OFF" device=""/>
-<part name="JP3" library="SparkFun-Connectors" deviceset="M04" device="PTH"/>
 <part name="LOGO3" library="SparkFun-Aesthetics" deviceset="SFE_LOGO_FLAME" device=".1_INCH"/>
 <part name="JP1" library="SparkFun-Connectors" deviceset="M03" device="PTH" value="UL"/>
 <part name="JP2" library="SparkFun-Connectors" deviceset="M03" device="PTH" value="UR"/>
-<part name="JP4" library="SparkFun-Connectors" deviceset="M03" device="PTH" value="LL"/>
-<part name="JP5" library="SparkFun-Connectors" deviceset="M03" device="PTH" value="LR"/>
-<part name="J1" library="SparkFun-Connectors" deviceset="RJ11-6" device="PTH"/>
-<part name="U$1" library="SparkFun-Connectors" deviceset="RJ45-8" device="PTH"/>
-<part name="JP6" library="SparkFun-Connectors" deviceset="M04" device="SCREW"/>
+<part name="JP3" library="SparkFun-Connectors" deviceset="M03" device="PTH" value="LL"/>
+<part name="JP4" library="SparkFun-Connectors" deviceset="M03" device="PTH" value="LR"/>
+<part name="FRAME1" library="SparkFun-Aesthetics" deviceset="FRAME-LETTER" device="">
+<attribute name="DESIGNER" value="N. Seidle"/>
+</part>
+<part name="JP5" library="SparkFun-Connectors" deviceset="M05" device="PTH"/>
 </parts>
 <sheets>
 <sheet>
 <plain>
-<text x="118.364" y="136.398" size="1.778" layer="97" rot="R270">E+</text>
-<text x="120.904" y="136.398" size="1.778" layer="97" rot="R270">E-</text>
-<text x="123.444" y="136.398" size="1.778" layer="97" rot="R270">A-</text>
-<text x="125.984" y="136.398" size="1.778" layer="97" rot="R270">A+</text>
-<text x="118.364" y="146.558" size="1.778" layer="97" rot="R270">Red</text>
-<text x="120.904" y="146.558" size="1.778" layer="97" rot="R270">Black</text>
-<text x="123.444" y="146.558" size="1.778" layer="97" rot="R270">White</text>
-<text x="125.984" y="146.558" size="1.778" layer="97" rot="R270">Green</text>
-<text x="172.72" y="10.16" size="1.778" layer="97">N. Seidle</text>
+<text x="120.396" y="132.842" size="1.778" layer="97" rot="R90">E+</text>
+<text x="122.936" y="132.842" size="1.778" layer="97" rot="R90">E-</text>
+<text x="125.476" y="132.842" size="1.778" layer="97" rot="R90">A-</text>
+<text x="128.016" y="132.842" size="1.778" layer="97" rot="R90">A+</text>
+<text x="120.396" y="143.002" size="1.778" layer="97" rot="R90">Red</text>
+<text x="122.936" y="143.002" size="1.778" layer="97" rot="R90">Black</text>
+<text x="125.476" y="143.002" size="1.778" layer="97" rot="R90">White</text>
+<text x="128.016" y="143.002" size="1.778" layer="97" rot="R90">Green</text>
 <text x="147.32" y="68.58" size="1.778" layer="97">Lower Right</text>
 <text x="101.6" y="68.58" size="1.778" layer="97">Upper Right</text>
 <text x="124.46" y="68.58" size="1.778" layer="97">Lower Left</text>
 <text x="78.74" y="68.58" size="1.778" layer="97">Upper Left</text>
-<text x="107.696" y="60.198" size="1.778" layer="97">3-Wire Load Sensors</text>
-<text x="106.172" y="62.992" size="1.778" layer="97">Common Bathroom Scale</text>
+<text x="106.68" y="60.96" size="1.778" layer="97">3-Wire Load Sensors</text>
+<text x="105.41" y="63.754" size="1.778" layer="97">Common Bathroom Scale</text>
 <text x="81.534" y="128.016" size="1.778" layer="97">Connection to Amplifier</text>
 <text x="75.692" y="82.804" size="1.778" layer="97">BLK</text>
 <text x="75.946" y="85.598" size="1.778" layer="97">WHT</text>
 <text x="75.946" y="88.138" size="1.778" layer="97">RED</text>
+<text x="83.82" y="53.34" size="2.032" layer="97">4 load sensors combine to create one load cell</text>
+<text x="130.556" y="132.842" size="1.778" layer="97" rot="R90">Shield</text>
+<text x="130.556" y="143.002" size="1.778" layer="97" rot="R90">Yellow</text>
+<text x="134.62" y="119.38" size="1.778" layer="97">Intentionally not-connected
+to create telescoping shield.</text>
 </plain>
 <instances>
-<instance part="FRAME1" gate="G$1" x="0" y="0"/>
-<instance part="FRAME1" gate="G$2" x="147.32" y="0"/>
 <instance part="U$7" gate="G$1" x="132.08" y="12.7"/>
 <instance part="STANDOFF1" gate="G$1" x="243.84" y="38.1"/>
@@
 <instance part="STANDOFF3" gate="G$1" x="233.68" y="38.1"/>
 <instance part="STANDOFF4" gate="G$1" x="228.6" y="38.1"/>
-<instance part="JP3" gate="G$1" x="121.92" y="127" rot="R270"/>
 <instance part="LOGO3" gate="G$1" x="109.22" y="5.08"/>
 <instance part="JP1" gate="G$1" x="83.82" y="86.36"/>
 <instance part="JP2" gate="G$1" x="106.68" y="86.36"/>
-<instance part="JP4" gate="G$1" x="129.54" y="86.36"/>
-<instance part="JP5" gate="G$1" x="152.4" y="86.36"/>
-<instance part="J1" gate="G$1" x="40.64" y="101.6"/>
-<instance part="U$1" gate="G$1" x="66.04" y="68.58"/>
-<instance part="JP6" gate="G$1" x="58.42" y="99.06"/>
+<instance part="JP3" gate="G$1" x="129.54" y="86.36"/>
+<instance part="JP4" gate="G$1" x="152.4" y="86.36"/>
+<instance part="FRAME1" gate="G$1" x="0" y="0">
+<attribute name="DESIGNER" x="0" y="0" size="1.27" layer="96" display="off"/>
+<attribute name="VERSION" x="0" y="0" size="1.27" layer="96" display="off"/>
+</instance>
+<instance part="FRAME1" gate="V" x="147.32" y="0"/>
+<instance part="JP5" gate="G$1" x="124.46" y="129.54" rot="R270"/>
 </instances>
 <busses>
@@
 <net name="N$1" class="0">
 <segment>
-<pinref part="JP5" gate="G$1" pin="1"/>
+<pinref part="JP4" gate="G$1" pin="1"/>
 <wire x1="160.02" y1="83.82" x2="162.56" y2="83.82" width="0.1524" layer="91"/>
 <wire x1="162.56" y1="83.82" x2="162.56" y2="76.2" width="0.1524" layer="91"/>
@@
 <net name="N$2" class="0">
 <segment>
-<pinref part="JP4" gate="G$1" pin="1"/>
+<pinref part="JP3" gate="G$1" pin="1"/>
 <wire x1="137.16" y1="83.82" x2="139.7" y2="83.82" width="0.1524" layer="91"/>
 <wire x1="139.7" y1="83.82" x2="139.7" y2="73.66" width="0.1524" layer="91"/>
@@
 <net name="N$3" class="0">
 <segment>
-<pinref part="JP5" gate="G$1" pin="2"/>
+<pinref part="JP4" gate="G$1" pin="2"/>
 <wire x1="160.02" y1="86.36" x2="165.1" y2="86.36" width="0.1524" layer="91"/>
 <wire x1="165.1" y1="86.36" x2="165.1" y2="96.52" width="0.1524" layer="91"/>
 <wire x1="165.1" y1="96.52" x2="142.24" y2="96.52" width="0.1524" layer="91"/>
 <wire x1="142.24" y1="96.52" x2="142.24" y2="86.36" width="0.1524" layer="91"/>
-<pinref part="JP4" gate="G$1" pin="2"/>
+<pinref part="JP3" gate="G$1" pin="2"/>
 <wire x1="142.24" y1="86.36" x2="137.16" y2="86.36" width="0.1524" layer="91"/>
 </segment>
@@
 <net name="E+" class="0">
 <segment>
-<pinref part="JP5" gate="G$1" pin="3"/>
+<pinref part="JP4" gate="G$1" pin="3"/>
 <wire x1="160.02" y1="88.9" x2="162.56" y2="88.9" width="0.1524" layer="91"/>
 <wire x1="162.56" y1="88.9" x2="162.56" y2="111.76" width="0.1524" layer="91"/>
 <wire x1="119.38" y1="111.76" x2="162.56" y2="111.76" width="0.1524" layer="91"/>
-<pinref part="JP3" gate="G$1" pin="1"/>
 <wire x1="119.38" y1="111.76" x2="119.38" y2="121.92" width="0.1524" layer="91"/>
+<pinref part="JP5" gate="G$1" pin="1"/>
 </segment>
 </net>
 <net name="A+" class="0">
 <segment>
-<wire x1="127" y1="109.22" x2="139.7" y2="109.22" width="0.1524" layer="91"/>
-<wire x1="139.7" y1="109.22" x2="139.7" y2="88.9" width="0.1524" layer="91"/>
-<pinref part="JP4" gate="G$1" pin="3"/>
+<wire x1="124.46" y1="106.68" x2="139.7" y2="106.68" width="0.1524" layer="91"/>
+<wire x1="139.7" y1="106.68" x2="139.7" y2="88.9" width="0.1524" layer="91"/>
+<pinref part="JP3" gate="G$1" pin="3"/>
 <wire x1="139.7" y1="88.9" x2="137.16" y2="88.9" width="0.1524" layer="91"/>
-<pinref part="JP3" gate="G$1" pin="4"/>
-<wire x1="127" y1="121.92" x2="127" y2="109.22" width="0.1524" layer="91"/>
+<wire x1="124.46" y1="106.68" x2="124.46" y2="121.92" width="0.1524" layer="91"/>
+<pinref part="JP5" gate="G$1" pin="3"/>
 </segment>
 </net>
@@
 <wire x1="114.3" y1="88.9" x2="116.84" y2="88.9" width="0.1524" layer="91"/>
 <wire x1="116.84" y1="88.9" x2="116.84" y2="109.22" width="0.1524" layer="91"/>
-<wire x1="116.84" y1="109.22" x2="124.46" y2="109.22" width="0.1524" layer="91"/>
-<pinref part="JP3" gate="G$1" pin="3"/>
-<wire x1="124.46" y1="109.22" x2="124.46" y2="121.92" width="0.1524" layer="91"/>
+<wire x1="116.84" y1="109.22" x2="127" y2="109.22" width="0.1524" layer="91"/>
+<wire x1="127" y1="121.92" x2="127" y2="109.22" width="0.1524" layer="91"/>
+<pinref part="JP5" gate="G$1" pin="4"/>
 </segment>
 </net>
 <net name="E-" class="0">
 <segment>
-<pinref part="JP3" gate="G$1" pin="2"/>
 <wire x1="121.92" y1="114.3" x2="121.92" y2="121.92" width="0.1524" layer="91"/>
 <wire x1="121.92" y1="114.3" x2="93.98" y2="114.3" width="0.1524" layer="91"/>
@@
 <pinref part="JP1" gate="G$1" pin="3"/>
 <wire x1="93.98" y1="88.9" x2="91.44" y2="88.9" width="0.1524" layer="91"/>
+<pinref part="JP5" gate="G$1" pin="2"/>
 </segment>
 </net>
@@
 </schematic>
 </drawing>
+<compatibility>
+<note version="6.3" minversion="6.2.2" severity="warning">
+Since Version 6.2.2 text objects can contain more than one line,
+which will not be processed correctly with this version.
+</note>
+</compatibility>
 </eagle>
